File: Prototype/Headphone Amplifier.sch (EAGLE design)
At the start: 28 parts, among them CN1 Input, CN2 Output, CN3 Power, Q1 BC547, Q2 BC559, Q3 BC559, Q4 BC547, Q5 BD140, Q6 BD139, Q7 BC547

Commit message: Renumbered the reference designators in the schematic
Parts:
- C1: value 4u7 -> 100n; device innove-passives:CPOL-E1.8-4 -> innove-passives:C5.0-2.5X7.5
- C2: value 100n -> 470u; device innove-passives:C5.0-2.5X7.5 -> innove-passives:CPOL-E5-10
- C3: value 470u -> 4u7; device innove-passives:CPOL-E5-10 -> innove-passives:CPOL-E1.8-4
- C4: value 1000u -> 10p; device innove-passives:CPOL-E5-10 -> innove-passives:C5.0-2.5X7.5
- C5: value 10p -> 1000u; device innove-passives:C5.0-2.5X7.5 -> innove-passives:CPOL-E5-10
- CN1: value Input -> Power
- CN2: value Output -> Input
- CN3: value Power -> Output
- Q1: value BC547 -> BC559; device innove-bjts:BC547 -> innove-bjts:BC559
- Q3: value BC559 -> BC547; device innove-bjts:BC559 -> innove-bjts:BC547
- Q5: value BD140 -> BC547; device innove-bjts:BD140 -> innove-bjts:BC547
- Q6: value BD139 -> BD140; device innove-bjts:BD139 -> innove-bjts:BD140
- Q7: value BC547 -> BD139; device innove-bjts:BC547 -> innove-bjts:BD139
- R1: value 6k8 -> 1k
- R10: value 68k -> 4k7
- R11: value 100k -> 10
- R12: value 1k -> 100k
- R2: value 10k -> 100k
- R3: value 1k -> 10k
- R4: value 100k -> 10k
- R5: value 10k -> 6k8
- R6: value 330 -> 1k
- R7: value 1k -> 330
- R8: value 4k7 -> 68k
- R9: value 10 -> 1k
Connections:
- net +3V3: now also C1.1, C2.+, CN1.1, Q1.E, Q6.E, R1.2, R10.2, R9.2; no longer C2.1, C3.+, CN3.1, Q3.E, Q5.E, R12.2, R6.2, R8.2
- net DCOUTPUT: now also C4.1, C5.+, Q7.C, R8.2; no longer C4.+, C5.1, Q5.C, R10.2
- net GND: now also C1.2, C2.-, Q3.E, Q5.E, R12.1, R2.1, R6.1; no longer C2.2, C3.-, Q1.E, Q7.E, R3.1, R5.1, R9.1
- net INPUT: now also C3.-, CN2.1, R2.2; no longer C1.-, CN1.1, R4.2
- net INTSTAGE: now also Q3.C; no longer Q1.C
- net N$1: now also R5.1, R6.2; no longer R1.1, R3.2
- net N$2: now also C3.+, R3.1; no longer C1.+, R2.1
- net N$3: now also R1.1; no longer R12.1
- net N$4: now also Q1.C, R4.2; no longer Q3.C, R5.2
- net N$5: now also Q1.B, R7.1; no longer Q3.B, R6.1
- net N$6: now also Q6.B, R9.1; no longer Q5.B, R7.1
- net N$8: now also Q5.C, Q7.B, R10.1; no longer Q6.B, Q7.C, R8.1
- net N$9: now also Q5.B, Q7.E, R11.2; no longer Q6.E, Q7.B, R9.2
- net NFB: now also C4.2, Q3.B, R3.2, R5.2, R8.1; no longer C5.2, Q1.B, R1.2, R10.1, R2.2
- net OUTPUT: now also C5.-, CN3.1, R12.2; no longer C4.-, CN2.1, R11.2
Other:
- moved on the sheet: C3, CN1, CN2, CN3, Q7, R1, R10, R11, R12, R2, R3, R4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

Commit message: Prototype circuit done
Connections:
- net +3V3 renamed +12V
Changed lines of the file:
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@@
 <instance part="GND7" gate="1" x="106.68" y="96.52"/>
 <instance part="+12V6" gate="G$1" x="116.84" y="134.62"/>
-<instance part="+12V5" gate="G$1" x="106.68" y="127"/>
+<instance part="+12V5" gate="G$1" x="106.68" y="129.54"/>
 <instance part="C1" gate="G$1" x="43.18" y="149.86"/>
 <instance part="+12V2" gate="G$1" x="43.18" y="157.48"/>
@@
 </segment>
 </net>
-<net name="+3V3" class="0">
-<segment>
-<pinref part="R7" gate="G$1" pin="2"/>
-<pinref part="+12V6" gate="G$1" pin="+3V3"/>
-</segment>
-<segment>
-<pinref part="Q1" gate="G$1" pin="E"/>
-<pinref part="+12V5" gate="G$1" pin="+3V3"/>
-</segment>
-<segment>
-<pinref part="C1" gate="G$1" pin="1"/>
-<pinref part="+12V2" gate="G$1" pin="+3V3"/>
-<wire x1="43.18" y1="152.4" x2="43.18" y2="154.94" width="0.1524" layer="91"/>
-</segment>
-<segment>
-<pinref part="C2" gate="G$1" pin="+"/>
-<pinref part="+12V3" gate="G$1" pin="+3V3"/>
-<wire x1="53.34" y1="152.4" x2="53.34" y2="154.94" width="0.1524" layer="91"/>
-</segment>
-<segment>
-<pinref part="R9" gate="G$1" pin="2"/>
-<pinref part="+12V7" gate="G$1" pin="+3V3"/>
-</segment>
-<segment>
-<pinref part="Q6" gate="G$1" pin="E"/>
-<pinref part="+12V9" gate="G$1" pin="+3V3"/>
-<wire x1="162.56" y1="114.3" x2="162.56" y2="111.76" width="0.1524" layer="91"/>
-</segment>
-<segment>
-<pinref part="R10" gate="G$1" pin="2"/>
-<pinref part="+12V8" gate="G$1" pin="+3V3"/>
-</segment>
-<segment>
-<pinref part="CN1" gate="G$1" pin="1"/>
-<pinref part="+12V1" gate="G$1" pin="+3V3"/>
-<wire x1="25.4" y1="149.86" x2="33.02" y2="149.86" width="0.1524" layer="91"/>
-<wire x1="33.02" y1="149.86" x2="33.02" y2="154.94" width="0.1524" layer="91"/>
-</segment>
-<segment>
-<pinref part="R1" gate="G$1" pin="2"/>
-<pinref part="+12V4" gate="G$1" pin="+3V3"/>
-</segment>
-</net>
 <net name="N$4" class="0">
 <segment>
@@
 </segment>
 </net>
+<net name="+12V" class="0">
+<segment>
+<pinref part="C2" gate="G$1" pin="+"/>
+<pinref part="+12V3" gate="G$1" pin="+12V"/>
+<wire x1="53.34" y1="152.4" x2="53.34" y2="154.94" width="0.1524" layer="91"/>
+</segment>
+<segment>
+<pinref part="R7" gate="G$1" pin="2"/>
+<pinref part="+12V6" gate="G$1" pin="+12V"/>
+</segment>
+<segment>
+<pinref part="Q1" gate="G$1" pin="E"/>
+<pinref part="+12V5" gate="G$1" pin="+12V"/>
+<wire x1="106.68" y1="127" x2="106.68" y2="124.46" width="0.1524" layer="91"/>
+</segment>
+<segment>
+<pinref part="C1" gate="G$1" pin="1"/>
+<pinref part="+12V2" gate="G$1" pin="+12V"/>
+<wire x1="43.18" y1="152.4" x2="43.18" y2="154.94" width="0.1524" layer="91"/>
+</segment>
+<segment>
+<pinref part="R9" gate="G$1" pin="2"/>
+<pinref part="+12V7" gate="G$1" pin="+12V"/>
+</segment>
+<segment>
+<pinref part="Q6" gate="G$1" pin="E"/>
+<pinref part="+12V9" gate="G$1" pin="+12V"/>
+<wire x1="162.56" y1="114.3" x2="162.56" y2="111.76" width="0.1524" layer="91"/>
+</segment>
+<segment>
+<pinref part="R10" gate="G$1" pin="2"/>
+<pinref part="+12V8" gate="G$1" pin="+12V"/>
+</segment>
+<segment>
+<pinref part="CN1" gate="G$1" pin="1"/>
+<pinref part="+12V1" gate="G$1" pin="+12V"/>
+<wire x1="25.4" y1="149.86" x2="33.02" y2="149.86" width="0.1524" layer="91"/>
+<wire x1="33.02" y1="149.86" x2="33.02" y2="154.94" width="0.1524" layer="91"/>
+</segment>
+<segment>
+<pinref part="R1" gate="G$1" pin="2"/>
+<pinref part="+12V4" gate="G$1" pin="+12V"/>
+</segment>
+</net>
