File: Prototype/Shunt Regulator.sch (EAGLE design)
At the start: 21 parts, among them Q1 BC547, Q2 BC559, Q3 TIP32, Q4 TIP32, Q5 BC559, Q6 BC559

Commit message: Finished the shunt regulator prototype
Parts:
- C2: value 1000u -> 100u; device innove-passives:CPOL-E5-10 -> innove-passives:CPOL-E2.5-6
- Q1: value BC547 -> BC559; device innove-bjts:BC547 -> innove-bjts:BC559
- Q2, Q6: value BC559 -> TIP32; device innove-bjts:BC559 -> innove-bjts:TIP32
- Q3, Q4: value TIP32 -> BC559; device innove-bjts:TIP32 -> innove-bjts:BC559
- Q5: value BC559 -> BC547; device innove-bjts:BC559 -> innove-bjts:BC547
- R3: value 220 -> 10k
- R4: value 10k -> 220
Connections:
- removed net N$3: C4.+, C5.+, CN2.1, CN3.1, JP1.2, Q4.C, Q5.E, R3.2, R5.A
- new net OUTPUT: C4.+, C5.+, CN2.1, CN3.1, JP1.2, Q2.C, Q3.E, R4.2, R5.A
- net +15V: now also Q1.E; no longer Q2.E
- net GND: now also Q6.C, R3.1; no longer Q3.C, R4.1
- net N$1: now also Q1.C, Q2.B; no longer Q2.C, Q4.B
- net N$2: now also Q1.B, Q2.E; no longer Q2.B, Q4.E
- net N$4: now also Q4.C, Q5.C, Q6.B; no longer Q1.C, Q3.B, Q6.C
- net N$5: now also Q3.B, Q4.E, R4.1; no longer Q5.B, Q6.E, R3.1
- net N$6: now also Q3.C, Q4.B, R3.2; no longer Q5.C, Q6.B, R4.2
- net N$7: now also Q5.E; no longer Q1.E
- net N$8: now also Q5.B; no longer Q1.B
- net N$9: now also Q6.E; no longer Q3.E
Other:
- moved on the sheet: Q2, Q3, Q4, Q6, R3, R4
Changed lines of the file:
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@@
 <part name="+15V3" library="innove-supply" deviceset="+15V" device=""/>
 <part name="GND3" library="innove-supply" deviceset="GND" device=""/>
-<part name="Q1" library="innove-bjts" deviceset="BC547" device=""/>
-<part name="Q2" library="innove-bjts" deviceset="BC559" device=""/>
-<part name="Q4" library="innove-bjts" deviceset="TIP32" device=""/>
+<part name="Q5" library="innove-bjts" deviceset="BC547" device=""/>
+<part name="Q1" library="innove-bjts" deviceset="BC559" device=""/>
+<part name="Q2" library="innove-bjts" deviceset="TIP32" device=""/>
 <part name="R1" library="innove-passives" deviceset="R" device="T0207" value="4k7"/>
 <part name="R2" library="innove-passives" deviceset="R" device="T0207" value="6R8"/>
+<part name="+15V5" library="innove-supply" deviceset="+15V" device=""/>
 <part name="+15V4" library="innove-supply" deviceset="+15V" device=""/>
-<part name="+15V5" library="innove-supply" deviceset="+15V" device=""/>
 <part name="GND4" library="innove-supply" deviceset="GND" device=""/>
-<part name="Q5" library="innove-bjts" deviceset="BC559" device=""/>
-<part name="Q6" library="innove-bjts" deviceset="BC559" device=""/>
-<part name="R3" library="innove-passives" deviceset="R" device="T0207" value="220"/>
-<part name="R4" library="innove-passives" deviceset="R" device="T0207" value="10k"/>
+<part name="Q3" library="innove-bjts" deviceset="BC559" device=""/>
+<part name="Q4" library="innove-bjts" deviceset="BC559" device=""/>
+<part name="R4" library="innove-passives" deviceset="R" device="T0207" value="220"/>
+<part name="R3" library="innove-passives" deviceset="R" device="T0207" value="10k"/>
 <part name="GND5" library="innove-supply" deviceset="GND" device=""/>
-<part name="Q3" library="innove-bjts" deviceset="TIP32" device=""/>
+<part name="Q6" library="innove-bjts" deviceset="TIP32" device=""/>
 <part name="LED1" library="innove-leds" deviceset="LED" device="5MM" value="Red"/>
 <part name="C3" library="innove-passives" deviceset="CPOL" device="-E5-10" value="1000u"/>
 <part name="GND6" library="innove-supply" deviceset="GND" device=""/>
 <part name="GND7" library="innove-supply" deviceset="GND" device=""/>
-<part name="C2" library="innove-passives" deviceset="CPOL" device="-E5-10" value="1000u"/>
 <part name="C4" library="innove-passives" deviceset="CPOL" device="-E2.5-6" value="100u"/>
 <part name="R5" library="rcl" deviceset="R-TRIMM" device="3296Y" value="100k"/>
@@
 <part name="GND11" library="innove-supply" deviceset="GND" device=""/>
 <part name="GND12" library="innove-supply" deviceset="GND" device=""/>
+<part name="C2" library="innove-passives" deviceset="CPOL" device="-E2.5-6" value="100u"/>
 </parts>
 <sheets>
@@
 <instance part="+15V3" gate="G$1" x="53.34" y="154.94"/>
 <instance part="GND3" gate="1" x="53.34" y="137.16"/>
-<instance part="Q1" gate="G$1" x="114.3" y="55.88" rot="MR0"/>
-<instance part="Q2" gate="G$1" x="93.98" y="127" rot="MR0"/>
-<instance part="Q4" gate="G$1" x="99.06" y="116.84"/>
+<instance part="Q5" gate="G$1" x="114.3" y="55.88" rot="MR0"/>
+<instance part="Q1" gate="G$1" x="93.98" y="127" rot="MR0"/>
+<instance part="Q2" gate="G$1" x="99.06" y="116.84"/>
 <instance part="R1" gate="G$1" x="91.44" y="106.68" rot="R90"/>
 <instance part="R2" gate="G$1" x="101.6" y="137.16" rot="R90"/>
-<instance part="+15V4" gate="G$1" x="101.6" y="144.78"/>
-<instance part="+15V5" gate="G$1" x="91.44" y="137.16"/>
+<instance part="+15V5" gate="G$1" x="101.6" y="144.78"/>
+<instance part="+15V4" gate="G$1" x="91.44" y="137.16"/>
 <instance part="GND4" gate="1" x="91.44" y="99.06"/>
-<instance part="Q5" gate="G$1" x="104.14" y="88.9" rot="MR0"/>
-<instance part="Q6" gate="G$1" x="109.22" y="78.74"/>
-<instance part="R3" gate="G$1" x="111.76" y="99.06" rot="R90"/>
-<instance part="R4" gate="G$1" x="101.6" y="68.58" rot="R90"/>
+<instance part="Q3" gate="G$1" x="104.14" y="88.9" rot="MR0"/>
+<instance part="Q4" gate="G$1" x="109.22" y="78.74"/>
+<instance part="R4" gate="G$1" x="111.76" y="99.06" rot="R90"/>
+<instance part="R3" gate="G$1" x="101.6" y="68.58" rot="R90"/>
 <instance part="GND5" gate="1" x="101.6" y="60.96"/>
-<instance part="Q3" gate="G$1" x="147.32" y="68.58"/>
+<instance part="Q6" gate="G$1" x="147.32" y="68.58"/>
 <instance part="LED1" gate="G$1" x="106.68" y="43.18"/>
 <instance part="C3" gate="G$1" x="116.84" y="43.18"/>
 <instance part="GND6" gate="1" x="106.68" y="35.56"/>
 <instance part="GND7" gate="1" x="116.84" y="35.56"/>
-<instance part="C2" gate="G$1" x="53.34" y="147.32"/>
 <instance part="C4" gate="G$1" x="124.46" y="88.9"/>
 <instance part="R5" gate="G$1" x="137.16" y="55.88" rot="R180"/>
@@
 <instance part="GND11" gate="1" x="180.34" y="96.52"/>
 <instance part="GND12" gate="1" x="180.34" y="71.12"/>
+<instance part="C2" gate="G$1" x="53.34" y="147.32"/>
 </instances>
 <busses>
@@
 </segment>
 <segment>
-<pinref part="R4" gate="G$1" pin="1"/>
+<pinref part="R3" gate="G$1" pin="1"/>
 <pinref part="GND5" gate="1" pin="GND"/>
 </segment>
@@
 <segment>
 <pinref part="GND9" gate="1" pin="GND"/>
-<pinref part="Q3" gate="G$1" pin="C"/>
+<pinref part="Q6" gate="G$1" pin="C"/>
 <wire x1="149.86" y1="60.96" x2="149.86" y2="63.5" width="0.1524" layer="91"/>
 </segment>
@@
 <segment>
 <pinref part="R2" gate="G$1" pin="2"/>
+<pinref part="+15V5" gate="G$1" pin="+15V"/>
+</segment>
+<segment>
+<pinref part="Q1" gate="G$1" pin="E"/>
 <pinref part="+15V4" gate="G$1" pin="+15V"/>
-</segment>
-<segment>
-<pinref part="Q2" gate="G$1" pin="E"/>
-<pinref part="+15V5" gate="G$1" pin="+15V"/>
 <wire x1="91.44" y1="134.62" x2="91.44" y2="132.08" width="0.1524" layer="91"/>
 </segment>
@@
 <segment>
 <pinref part="R1" gate="G$1" pin="2"/>
-<pinref part="Q2" gate="G$1" pin="C"/>
+<pinref part="Q1" gate="G$1" pin="C"/>
 <wire x1="91.44" y1="111.76" x2="91.44" y2="116.84" width="0.1524" layer="91"/>
-<pinref part="Q4" gate="G$1" pin="B"/>
+<pinref part="Q2" gate="G$1" pin="B"/>
 <wire x1="91.44" y1="116.84" x2="91.44" y2="121.92" width="0.1524" layer="91"/>
 <wire x1="96.52" y1="116.84" x2="91.44" y2="116.84" width="0.1524" layer="91"/>
@@
 <segment>
 <pinref part="R2" gate="G$1" pin="1"/>
-<pinref part="Q2" gate="G$1" pin="B"/>
+<pinref part="Q1" gate="G$1" pin="B"/>
 <wire x1="101.6" y1="127" x2="101.6" y2="132.08" width="0.1524" layer="91"/>
 <wire x1="96.52" y1="127" x2="101.6" y2="127" width="0.1524" layer="91"/>
-<pinref part="Q4" gate="G$1" pin="E"/>
+<pinref part="Q2" gate="G$1" pin="E"/>
 <wire x1="101.6" y1="121.92" x2="101.6" y2="127" width="0.1524" layer="91"/>
 <junction x="101.6" y="127"/>
 </segment>
 </net>
-<net name="N$3" class="0">
-<segment>
-<pinref part="Q4" gate="G$1" pin="C"/>
+<net name="OUTPUT" class="0">
+<segment>
+<pinref part="Q2" gate="G$1" pin="C"/>
 <wire x1="101.6" y1="111.76" x2="101.6" y2="106.68" width="0.1524" layer="91"/>
-<pinref part="Q5" gate="G$1" pin="E"/>
+<pinref part="Q3" gate="G$1" pin="E"/>
 <wire x1="101.6" y1="106.68" x2="101.6" y2="104.14" width="0.1524" layer="91"/>
 <wire x1="101.6" y1="93.98" x2="101.6" y2="106.68" width="0.1524" layer="91"/>
-<pinref part="R3" gate="G$1" pin="2"/>
+<pinref part="R4" gate="G$1" pin="2"/>
 <wire x1="101.6" y1="106.68" x2="111.76" y2="106.68" width="0.1524" layer="91"/>
 <wire x1="111.76" y1="106.68" x2="111.76" y2="104.14" width="0.1524" layer="91"/>
@@
 <net name="N$5" class="0">
 <segment>
-<pinref part="R3" gate="G$1" pin="1"/>
-<pinref part="Q6" gate="G$1" pin="E"/>
+<pinref part="R4" gate="G$1" pin="1"/>
+<pinref part="Q4" gate="G$1" pin="E"/>
 <wire x1="111.76" y1="93.98" x2="111.76" y2="88.9" width="0.1524" layer="91"/>
-<pinref part="Q5" gate="G$1" pin="B"/>
+<pinref part="Q3" gate="G$1" pin="B"/>
 <wire x1="111.76" y1="88.9" x2="111.76" y2="83.82" width="0.1524" layer="91"/>
 <wire x1="106.68" y1="88.9" x2="111.76" y2="88.9" width="0.1524" layer="91"/>
@@
 <net name="N$6" class="0">
 <segment>
-<pinref part="Q5" gate="G$1" pin="C"/>
+<pinref part="Q3" gate="G$1" pin="C"/>
 <wire x1="101.6" y1="83.82" x2="101.6" y2="78.74" width="0.1524" layer="91"/>
-<pinref part="Q6" gate="G$1" pin="B"/>
+<pinref part="Q4" gate="G$1" pin="B"/>
 <wire x1="101.6" y1="78.74" x2="106.68" y2="78.74" width="0.1524" layer="91"/>
-<pinref part="R4" gate="G$1" pin="2"/>
+<pinref part="R3" gate="G$1" pin="2"/>
 <wire x1="101.6" y1="73.66" x2="101.6" y2="78.74" width="0.1524" layer="91"/>
 <junction x="101.6" y="78.74"/>
@@
 <net name="N$4" class="0">
 <segment>
-<pinref part="Q3" gate="G$1" pin="B"/>
-<pinref part="Q6" gate="G$1" pin="C"/>
+<pinref part="Q6" gate="G$1" pin="B"/>
+<pinref part="Q4" gate="G$1" pin="C"/>
 <wire x1="144.78" y1="68.58" x2="111.76" y2="68.58" width="0.1524" layer="91"/>
 <wire x1="111.76" y1="68.58" x2="111.76" y2="73.66" width="0.1524" layer="91"/>
-<pinref part="Q1" gate="G$1" pin="C"/>
+<pinref part="Q5" gate="G$1" pin="C"/>
 <wire x1="111.76" y1="60.96" x2="111.76" y2="68.58" width="0.1524" layer="91"/>
 <junction x="111.76" y="68.58"/>
@@
 <wire x1="111.76" y1="48.26" x2="116.84" y2="48.26" width="0.1524" layer="91"/>
 <wire x1="116.84" y1="48.26" x2="116.84" y2="45.72" width="0.1524" layer="91"/>
-<pinref part="Q1" gate="G$1" pin="E"/>
+<pinref part="Q5" gate="G$1" pin="E"/>
 <wire x1="111.76" y1="50.8" x2="111.76" y2="48.26" width="0.1524" layer="91"/>
 <junction x="111.76" y="48.26"/>
@@
 <pinref part="C4" gate="G$1" pin="-"/>
 <wire x1="124.46" y1="83.82" x2="124.46" y2="55.88" width="0.1524" layer="91"/>
-<pinref part="Q1" gate="G$1" pin="B"/>
+<pinref part="Q5" gate="G$1" pin="B"/>
 <wire x1="124.46" y1="55.88" x2="116.84" y2="55.88" width="0.1524" layer="91"/>
 <pinref part="R5" gate="G$1" pin="S"/>
@@
 <segment>
 <pinref part="JP1" gate="A" pin="1"/>
-<pinref part="Q3" gate="G$1" pin="E"/>
+<pinref part="Q6" gate="G$1" pin="E"/>
 <wire x1="149.86" y1="81.28" x2="149.86" y2="73.66" width="0.1524" layer="91"/>
 </segment>
@@
 </sheet>
 </sheets>
+<errors>
+</errors>
 </schematic>
 </drawing>
